File: macropad.kicad_pcb (KiCad board)
At the start: 2 copper layers, 64.7 x 84.6 mm, 35 parts, among them J1 Conn_01x04_Socket, SW1 SW_Push, SW10 SW_Push, SW2 SW_Push, SW3 SW_Push, SW4 SW_Push, SW5 SW_Push, SW6 SW_Push, SW7 SW_Push, SW8 SW_Push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

Commit message: Add files via upload
Routing:
- net GND: track 38.7 -> 100.8 mm, vias 1 -> 3
- net col1: track 171.3 -> 180.8 mm
Changed lines of the file:
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@@
+	)
+	(segment
+		(start 141.661 99.391)
+		(end 141.661 102.307471)
+		(width 0.2)
+		(layer "F.Cu")
+		(net 2)
+	)
+	(segment
+		(start 141.59 99.32)
+		(end 141.661 99.391)
+		(width 0.2)
+		(layer "F.Cu")
+		(net 2)
+	)
+	(segment
+		(start 139.065 81.75)
+		(end 152.85 81.75)
+		(width 0.2)
+		(layer "F.Cu")
+		(net 2)
 	)
 	(segment
@@
 	)
 	(segment
+		(start 141.661 102.307471)
+		(end 133.333471 110.635)
+		(width 0.2)
+		(layer "F.Cu")
+		(net 2)
+	)
+	(segment
+		(start 133.333471 110.635)
+		(end 132.2 110.635)
+		(width 0.2)
+		(layer "F.Cu")
+		(net 2)
+	)
+	(segment
 		(start 169.31 67.5)
 		(end 168.27 67.5)
@@
 		(net 2)
 	)
+	(segment
+		(start 132.16 88.655)
+		(end 139.065 81.75)
+		(width 0.2)
+		(layer "F.Cu")
+		(net 2)
+	)
+	(via
+		(at 141.59 99.32)
+		(size 0.6)
+		(drill 0.3)
+		(layers "F.Cu" "B.Cu")
+		(net 2)
+	)
 	(via
 		(at 168.27 67.5)
+		(size 0.6)
+		(drill 0.3)
+		(layers "F.Cu" "B.Cu")
+		(net 2)
+	)
+	(via
+		(at 152.85 81.75)
 		(size 0.6)
 		(drill 0.3)
@@
 	)
 	(segment
+		(start 152.85 88.73382)
+		(end 142.26382 99.32)
+		(width 0.2)
+		(layer "B.Cu")
+		(net 2)
+	)
+	(segment
+		(start 142.26382 99.32)
+		(end 141.59 99.32)
+		(width 0.2)
+		(layer "B.Cu")
+		(net 2)
+	)
+	(segment
 		(start 145.482131 61.617)
 		(end 142.141131 64.958)
@@
 	)
 	(segment
+		(start 152.85 81.75)
+		(end 152.85 88.73382)
+		(width 0.2)
+		(layer "B.Cu")
+		(net 2)
+	)
+	(segment
 		(start 162.387 61.617)
 		(end 145.482131 61.617)
@@
 	)
 	(segment
+		(start 170.47 76.5)
+		(end 170.47 84.44)
+		(width 0.2)
+		(layer "F.Cu")
+		(net 29)
+	)
+	(segment
+		(start 171.59 75.38)
+		(end 170.47 76.5)
+		(width 0.2)
+		(layer "F.Cu")
+		(net 29)
+	)
+	(segment

Commit message: Add files via upload
Routing:
- net GND: track 100.8 -> 222.0 mm, vias 3 -> 5
- net +5V: track 213.5 -> 216.2 mm
