File: PCB/macropad.kicad_sch (KiCad schematic)
At the start: 29 parts, among them J1 Conn_01x04_Socket, SW1 SW_Push, SW10 SW_Push, SW2 SW_Push, SW3 SW_Push, SW4 SW_Push, SW5 SW_Push, SW6 SW_Push, SW7 SW_Push, SW8 SW_Push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

Commit message: Add files via upload
Parts:
- D1, D2, D3, D4, D5, D6: footprint LED_SMD:LED_SK6812MINI_PLCC4_3.5x3.5mm_P1.75mm -> led's:SK6812MINI-E_fixed
Changed lines of the file:
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@@
 			)
 		)
-		(property "Footprint" "LED_SMD:LED_SK6812MINI_PLCC4_3.5x3.5mm_P1.75mm"
+		(property "Footprint" "led's:SK6812MINI-E_fixed"
 			(at 153.67 130.81 0)
 			(effects
@@
 			)
 		)
-		(property "Footprint" "LED_SMD:LED_SK6812MINI_PLCC4_3.5x3.5mm_P1.75mm"
+		(property "Footprint" "led's:SK6812MINI-E_fixed"
 			(at 107.95 130.81 0)
 			(effects
@@
 			)
 		)
-		(property "Footprint" "LED_SMD:LED_SK6812MINI_PLCC4_3.5x3.5mm_P1.75mm"
+		(property "Footprint" "led's:SK6812MINI-E_fixed"
 			(at 92.71 130.81 0)
 			(effects
@@
 			)
 		)
-		(property "Footprint" "LED_SMD:LED_SK6812MINI_PLCC4_3.5x3.5mm_P1.75mm"
+		(property "Footprint" "led's:SK6812MINI-E_fixed"
 			(at 138.43 130.81 0)
 			(effects
@@
 			)
 		)
-		(property "Footprint" "LED_SMD:LED_SK6812MINI_PLCC4_3.5x3.5mm_P1.75mm"
+		(property "Footprint" "led's:SK6812MINI-E_fixed"
 			(at 123.19 130.81 0)
 			(effects
@@
 			)
 		)
-		(property "Footprint" "LED_SMD:LED_SK6812MINI_PLCC4_3.5x3.5mm_P1.75mm"
+		(property "Footprint" "led's:SK6812MINI-E_fixed"
 			(at 168.91 130.81 0)
 			(effects
